File: Drivers.kicad_sch (KiCad schematic)
At the start: 39 parts, among them U12 NSI8220, U4 NSI8220, U6 NSI8220

Commit message: VER1.0: составил список примерно 95% компонентов
Parts:
- added C124, C125, C126, C127, C128, C129, C130, C131: 100n, Capacitor_SMD:C_0805_2012Metric_Pad1.18x1.45mm_HandSolder, symbol Device:C_Small
- C100, C101, C102, C103, C31, C34, C89, C93, C96, C97: Description P/N (none) -> Capacitor SMD 25V
- C104, C105, C44, C88, C94, C95, C98, C99: Description P/N (none) -> Capacitor SMD 50V
- D10, D12, D17: value NSD1624 -> (none); Description P/N (none) -> Gate driver; Product Name (none) -> NSD1624
- D11, D16, D18: value D_Small -> (none); Description P/N (none) -> Ultrafast diode; Product Name (none) -> ES1D-E3/61T
- D19, D22: Description P/N (none) -> Gate driver; Product Name (none) -> NSI6602
- R52, R57, R60, R61, R62, R63, R64, R65, R66, R67: Description P/N (none) -> Resistor SMD 1%
- U12, U4, U6: value NSI8220 -> (none); Description P/N (none) -> Digital isolator; Product Name (none) -> NSI8220
Connections:
- net +3.3V: now also C124.2, C126.2, C128.2, C130.2, C131.2
- net +3.3VP: now also C125.2, C127.2, C129.2
- net GND: now also C124.1, C126.1, C128.1, C130.1, C131.1
- net GNDPWR: now also C125.1, C127.1, C129.1
