File: Nauka_DCAC.kicad_pcb (KiCad board)
At the start: 2 copper layers, 63 parts, among them Q1 WMK115N15HG2, Q2 WMK115N15HG2, Q3 WMK115N15HG2, Q4 WMK115N15HG2, Q5 WMK115N15HG2, Q6 WMK115N15HG2, Q7 WMK115N15HG2, Q8 WMK115N15HG2, U1 CH704150CT, U2 CH704150CT

Commit message: VER1.0: собрал силовую часть на схеме
Parts:
- removed C73, C76, C80, C83: 10u, Capacitor_SMD:C_1206_3216Metric_Pad1.33x1.80mm_HandSolder
- removed C74: 1u, Capacitor_SMD:C_1206_3216Metric_Pad1.33x1.80mm_HandSolder
- removed C75, C84, C85: 56p, Capacitor_SMD:C_0805_2012Metric_Pad1.18x1.45mm_HandSolder
- removed C77, C81: 2.2u, Capacitor_SMD:C_0805_2012Metric_Pad1.18x1.45mm_HandSolder
- removed C79, C82: 0.1u, Capacitor_SMD:C_0805_2012Metric_Pad1.18x1.45mm_HandSolder
- removed C86: 100n, Capacitor_SMD:C_0805_2012Metric_Pad1.18x1.45mm_HandSolder
- removed C87: 1n, Capacitor_SMD:C_0805_2012Metric_Pad1.18x1.45mm_HandSolder
- removed D32, D33: ~, LED_SMD:LED_1206_3216Metric_Pad1.42x1.75mm_HandSolder
- removed D34: ~, MORNSUN:WRB_S-3WR2
- removed D35, D38: ~, Package_TO_SOT_SMD:SOT-23
- removed D36: ~, Package_SO:SOIC-8_7.5x5.85mm_P1.27mm
- removed D37: ~, LED_SMD:LED_0805_2012Metric
- removed L13: 4.7u, Inductor_SMD:L_1812_4532Metric_Pad1.30x3.40mm_HandSolder
- removed R65: 10k, Resistor_SMD:R_1206_3216Metric_Pad1.30x1.75mm_HandSolder
- removed R66, R67, R68, R69: 110k, Resistor_SMD:R_1206_3216Metric
- removed R70: 11.3k, Resistor_SMD:R_1206_3216Metric
- removed R71: 120, Resistor_SMD:R_0805_2012Metric_Pad1.20x1.40mm_HandSolder
- removed R72, R73, R75, R76: 1k, Resistor_SMD:R_0805_2012Metric_Pad1.20x1.40mm_HandSolder
- removed R74: 750, Resistor_SMD:R_0805_2012Metric_Pad1.20x1.40mm_HandSolder
- removed R77: 510, Resistor_SMD:R_0805_2012Metric_Pad1.20x1.40mm_HandSolder
- removed U16: ~, Package_TO_SOT_SMD:SOT-23-5
- removed U32: ~, Package_TO_SOT_SMD:SOT-223-3_TabPin2
- added C1: 12p, Capacitor_SMD:C_0805_2012Metric_Pad1.18x1.45mm_HandSolder, F.Cu at (193.8, 70.8)
- added C10: 1u, Capacitor_SMD:C_0805_2012Metric_Pad1.18x1.45mm_HandSolder, F.Cu at (193.4, 117.7)
- added C11: 100n, Capacitor_SMD:C_0805_2012Metric_Pad1.18x1.45mm_HandSolder, F.Cu at (193.4, 120.7)
- added C12: 2.2u, Capacitor_THT:C_Rect_L31.5mm_W13.0mm_P27.50mm_MKS4, F.Cu at (198.2, 108.7)
- added C13: 470n, Capacitor_SMD:C_1206_3216Metric_Pad1.33x1.80mm_HandSolder, F.Cu at (198.2, 111.7)
- added C14: 1u, Capacitor_SMD:C_0805_2012Metric_Pad1.18x1.45mm_HandSolder, F.Cu at (198.2, 114.7)
- added C15: 100n, Capacitor_SMD:C_0805_2012Metric_Pad1.18x1.45mm_HandSolder, F.Cu at (198.2, 117.7)
- added C16: 56p, Capacitor_SMD:C_0805_2012Metric_Pad1.18x1.45mm_HandSolder, F.Cu at (198.2, 120.7)
- added C17: 2.2u, Capacitor_SMD:C_0805_2012Metric_Pad1.18x1.45mm_HandSolder, F.Cu at (203.0, 108.7)
- added C18: 100n, Capacitor_SMD:C_0805_2012Metric_Pad1.18x1.45mm_HandSolder, F.Cu at (203.0, 111.7)
- added C19: 10u, Capacitor_SMD:C_1206_3216Metric_Pad1.33x1.80mm_HandSolder, F.Cu at (203.0, 114.7)
- added C2: 12p, Capacitor_SMD:C_0805_2012Metric_Pad1.18x1.45mm_HandSolder, F.Cu at (229.5, 72.3)
- added C20: 2.2u, Capacitor_SMD:C_0805_2012Metric_Pad1.18x1.45mm_HandSolder, F.Cu at (203.0, 117.7)
- added C21: 100n, Capacitor_SMD:C_0805_2012Metric_Pad1.18x1.45mm_HandSolder, F.Cu at (229.5, 89.8)
- added C22: 10u, Capacitor_SMD:C_1206_3216Metric_Pad1.33x1.80mm_HandSolder, F.Cu at (250.2, 109.4)
- added C23: 2.2u, Capacitor_SMD:C_1206_3216Metric_Pad1.33x1.80mm_HandSolder, F.Cu at (250.2, 112.8)
- added C24: 2.2u, Capacitor_SMD:C_1206_3216Metric_Pad1.33x1.80mm_HandSolder, F.Cu at (250.2, 116.1)
- added C25: 56p, Capacitor_SMD:C_0805_2012Metric_Pad1.18x1.45mm_HandSolder, F.Cu at (250.2, 119.5)
- added C26: 56p, Capacitor_SMD:C_0805_2012Metric_Pad1.18x1.45mm_HandSolder, F.Cu at (193.8, 85.3)
- added C27: 2.2u, Capacitor_SMD:C_1206_3216Metric_Pad1.33x1.80mm_HandSolder, F.Cu at (193.8, 99.9)
- added C28: 2.2u, Capacitor_SMD:C_1206_3216Metric_Pad1.33x1.80mm_HandSolder, F.Cu at (180.0, 54.2)
- added C29: 1m, Capacitor_THT:CP_Radial_D16.0mm_P7.50mm, F.Cu at (180.0, 57.5)
- added C30: 1m, Capacitor_THT:CP_Radial_D16.0mm_P7.50mm, F.Cu at (197.0, 46.5)
- added C31: 10u, Capacitor_SMD:C_1206_3216Metric_Pad1.33x1.80mm_HandSolder, F.Cu at (180.0, 64.2)
- added C32: 100n, Capacitor_SMD:C_0805_2012Metric_Pad1.18x1.45mm_HandSolder, F.Cu at (223.0, 77.6)
- added C33: 1n, Capacitor_SMD:C_0805_2012Metric_Pad1.18x1.45mm_HandSolder, F.Cu at (223.0, 80.6)
- added C7: 470n, Capacitor_SMD:C_1206_3216Metric_Pad1.33x1.80mm_HandSolder, F.Cu at (193.4, 108.7)
- added C8: 2.2u, Capacitor_THT:C_Rect_L31.5mm_W13.0mm_P27.50mm_MKS4, F.Cu at (193.4, 111.7)
- added C9: 470n, Capacitor_SMD:C_1206_3216Metric_Pad1.33x1.80mm_HandSolder, F.Cu at (193.4, 114.7)
- added D1: ~, LED_SMD:LED_0805_2012Metric, F.Cu at (253.8, 104.8)
- added D2: ~, LED_SMD:LED_0805_2012Metric, F.Cu at (218.3, 77.6)
- added D3: ~, LED_SMD:LED_1206_3216Metric_Pad1.42x1.75mm_HandSolder, F.Cu at (222.5, 68.6)
- added D4: ~, LED_SMD:LED_1206_3216Metric_Pad1.42x1.75mm_HandSolder, F.Cu at (255.4, 109.3)
- added D5: ~, Package_TO_SOT_SMD:SOT-23, F.Cu at (255.4, 112.3)
- added D6: ~, Package_SO:SOIC-8_7.5x5.85mm_P1.27mm, F.Cu at (213.3, 63.2)
- added D7: K7805-500R3, MORNSUN:K78xx-500R3, F.Cu at (212.9, 73.1)
- added D8: ~, LED_SMD:LED_0805_2012Metric, F.Cu at (218.3, 80.6)
- added D9: ~, Package_TO_SOT_SMD:SOT-23, F.Cu at (222.7, 61.7)
- added Q10: WMK115N15HG2, Package_TO_SOT_THT:TO-220-3_Horizontal_TabUp, F.Cu at (238.8, 100.4)
- added Q9: WMK115N15HG2, Package_TO_SOT_THT:TO-220-3_Horizontal_TabUp, F.Cu at (227.3, 100.4)
- added R13: 10k, Resistor_SMD:R_0805_2012Metric_Pad1.20x1.40mm_HandSolder, F.Cu at (244.4, 65.0)
- added R14: 10k, Resistor_SMD:R_0805_2012Metric_Pad1.20x1.40mm_HandSolder, F.Cu at (244.4, 67.9)
- added R15: 10k, Resistor_SMD:R_0805_2012Metric_Pad1.20x1.40mm_HandSolder, F.Cu at (244.4, 70.9)
- added R16: 1k, Resistor_SMD:R_0805_2012Metric_Pad1.20x1.40mm_HandSolder, F.Cu at (244.4, 73.8)
- added R17: 10k, Resistor_SMD:R_0805_2012Metric_Pad1.20x1.40mm_HandSolder, F.Cu at (244.4, 76.8)
- added R18: 10k, Resistor_SMD:R_0805_2012Metric_Pad1.20x1.40mm_HandSolder, F.Cu at (244.4, 79.7)
- added R19: 10, Resistor_SMD:R_0805_2012Metric_Pad1.20x1.40mm_HandSolder, F.Cu at (244.4, 82.7)
- added R20: 10, Resistor_SMD:R_0805_2012Metric_Pad1.20x1.40mm_HandSolder, F.Cu at (244.4, 85.6)
- added R21: 1k, Resistor_SMD:R_0805_2012Metric_Pad1.20x1.40mm_HandSolder, F.Cu at (244.4, 88.6)
- added R22: 4.7, Resistor_SMD:R_0805_2012Metric_Pad1.20x1.40mm_HandSolder, F.Cu at (249.2, 65.0)
- added R23: 4.7, Resistor_SMD:R_0805_2012Metric_Pad1.20x1.40mm_HandSolder, F.Cu at (249.2, 67.9)
- added R24: 10k, Resistor_SMD:R_0805_2012Metric_Pad1.20x1.40mm_HandSolder, F.Cu at (249.2, 70.9)
- added R25: 10k, Resistor_SMD:R_0805_2012Metric_Pad1.20x1.40mm_HandSolder, F.Cu at (249.2, 73.8)
- added R26: 10, Resistor_SMD:R_0805_2012Metric_Pad1.20x1.40mm_HandSolder, F.Cu at (249.2, 76.8)
- added R27: 10, Resistor_SMD:R_0805_2012Metric_Pad1.20x1.40mm_HandSolder, F.Cu at (249.2, 79.7)
- added R28: 10k, Resistor_SMD:R_0805_2012Metric_Pad1.20x1.40mm_HandSolder, F.Cu at (249.2, 82.7)
- added R29: 4.7, Resistor_SMD:R_0805_2012Metric_Pad1.20x1.40mm_HandSolder, F.Cu at (249.2, 85.6)
- added R30: 4.7, Resistor_SMD:R_0805_2012Metric_Pad1.20x1.40mm_HandSolder, F.Cu at (249.2, 88.6)
- added R31: 10, Resistor_SMD:R_0805_2012Metric_Pad1.20x1.40mm_HandSolder, F.Cu at (253.9, 65.0)
- added R32: 10, Resistor_SMD:R_0805_2012Metric_Pad1.20x1.40mm_HandSolder, F.Cu at (253.9, 67.9)
- added R33: 4.7, Resistor_SMD:R_0805_2012Metric_Pad1.20x1.40mm_HandSolder, F.Cu at (253.9, 70.9)
- added R34: 4.7, Resistor_SMD:R_0805_2012Metric_Pad1.20x1.40mm_HandSolder, F.Cu at (253.9, 73.8)
- added R35: 2k, Resistor_SMD:R_0805_2012Metric_Pad1.20x1.40mm_HandSolder, F.Cu at (253.9, 76.8)
- added R36: 3k, Resistor_SMD:R_0805_2012Metric_Pad1.20x1.40mm_HandSolder, F.Cu at (253.9, 79.7)
- added R37: 10k, Resistor_SMD:R_1206_3216Metric_Pad1.30x1.75mm_HandSolder, F.Cu at (253.9, 82.7)
- added R38: 110k, Resistor_SMD:R_1206_3216Metric, F.Cu at (253.9, 85.6)
- added R39: 2k, Resistor_SMD:R_0805_2012Metric_Pad1.20x1.40mm_HandSolder, F.Cu at (253.9, 88.6)
- added R40: 3k, Resistor_SMD:R_0805_2012Metric_Pad1.20x1.40mm_HandSolder, F.Cu at (258.7, 65.0)
- added R41: 110k, Resistor_SMD:R_1206_3216Metric, F.Cu at (258.7, 67.9)
- added R42: 110k, Resistor_SMD:R_1206_3216Metric, F.Cu at (258.7, 70.9)
- added R43: 110k, Resistor_SMD:R_1206_3216Metric, F.Cu at (258.7, 73.8)
- added R44: 11.3k, Resistor_SMD:R_1206_3216Metric, F.Cu at (258.7, 76.8)
- added R45: 120, Resistor_SMD:R_0805_2012Metric_Pad1.20x1.40mm_HandSolder, F.Cu at (203.9, 61.0)
- added R46: 1k, Resistor_SMD:R_0805_2012Metric_Pad1.20x1.40mm_HandSolder, F.Cu at (203.9, 63.9)
- added R47: 1k, Resistor_SMD:R_0805_2012Metric_Pad1.20x1.40mm_HandSolder, F.Cu at (203.9, 66.9)
- added R48: 1k, Resistor_SMD:R_0805_2012Metric_Pad1.20x1.40mm_HandSolder, F.Cu at (203.9, 69.8)
- added R49: 1k, Resistor_SMD:R_0805_2012Metric_Pad1.20x1.40mm_HandSolder, F.Cu at (203.9, 72.8)
- added R50: 750, Resistor_SMD:R_0805_2012Metric_Pad1.20x1.40mm_HandSolder, F.Cu at (203.9, 75.7)
- added R51: 510, Resistor_SMD:R_0805_2012Metric_Pad1.20x1.40mm_HandSolder, F.Cu at (203.9, 78.7)
- added U3: CH704150CT, Sensor_Current:Allegro_CB_PFF, F.Cu at (212.7, 114.4)
- added U4: ~, Package_TO_SOT_SMD:SOT-223-3_TabPin2, F.Cu at (211.2, 80.3)
- added U5: ~, Package_TO_SOT_SMD:SOT-23-5, F.Cu at (222.1, 72.7)
- added Y1: 16M, Crystal:Crystal_SMD_SeikoEpson_FA238-4Pin_3.2x2.5mm, F.Cu at (255.8, 116.1)
- C4, C5: value 1u -> 2.2u
- C6: value 100n -> 2.2u; footprint Capacitor_SMD:C_0805_2012Metric_Pad1.18x1.45mm_HandSolder -> Capacitor_THT:C_Rect_L31.5mm_W13.0mm_P27.50mm_MKS4
- R10: value 3k -> 10
- R11: value 2k -> 4.7
- R12: value 3k -> 4.7
- R3, R4: value 10k -> 10
- R5, R6: value 10k -> 4.7
- R9: value 2k -> 10
- U1: value CH704150CT -> STM32F405RGTx; footprint Sensor_Current:Allegro_CB_PFF -> Package_QFP:LQFP-64_10x10mm_P0.5mm
Connections:
- C3 pad 1: +5V -> GND
- C3 pad 2: GND -> /NRST
- C4 pad 1: +5V -> Net-(U1-VCAP_1)
- C5 pad 1: +5V -> Net-(U1-VCAP_2)
- C6 pad 1: +5V -> Net-(Q1-D)
- C6 pad 2: GND -> GNDPWR
- Q1 pad 1: /GH4 -> /GH1
- Q1 pad 3: /Bat+ -> /A
- Q2 pad 1: /GL4 -> /GL1
- Q2 pad 2: /Bat+ -> /A
- Q3 pad 1: /GL3 -> /GH2
- Q3 pad 2: /C -> Net-(Q1-D)
- Q3 pad 3: GNDPWR -> /B
- Q4 pad 1: /GH3 -> /GL2
- Q4 pad 2: Net-(Q1-D) -> /B
- Q4 pad 3: /C -> GNDPWR
- Q5 pad 1: /GH2 -> /GH3
- Q5 pad 3: /B -> /C
- Q6 pad 1: /GL2 -> /GL3
- Q6 pad 2: /B -> /C
- Q7 pad 1: /GH1 -> /GH4
- Q7 pad 3: /A -> /S1
- Q8 pad 1: /GL1 -> /GH5
- Q8 pad 2: /A -> Net-(Q1-D)
- Q8 pad 3: GNDPWR -> /S2
- R1 pad 1: /GL1 -> /GH1
- R1 pad 2: GNDPWR -> /A
- R10 pad 1: /Current_A -> /GL2
- R10 pad 2: GND -> /GL2_ON
- R11 pad 1: Net-(U2-VIOUT) -> /GH2
- R11 pad 2: /Current_C -> /GH2_OFF
- R12 pad 1: /Current_C -> /GL2
- R12 pad 2: GND -> /GL2_OFF
- R2 pad 1: /GL2 -> /GL1
- R3 pad 1: /GL3 -> /GH1
- R3 pad 2: GNDPWR -> /GH1_ON
- R4 pad 1: /GL4 -> /GL1
- R4 pad 2: GNDPWR -> /GL1_ON
- R5 pad 2: /A -> /GH1_OFF
- R6 pad 1: /GH2 -> /GL1
- R6 pad 2: /B -> /GL1_OFF
- R7 pad 1: /GH3 -> /GH2
- R7 pad 2: /C -> /B
- R8 pad 1: /GH4 -> /GL2
- R8 pad 2: /Bat+ -> GNDPWR
- R9 pad 1: Net-(U1-VIOUT) -> /GH2
- R9 pad 2: /Current_A -> /GH2_ON
- U1 pad 1: +5V -> +3.3V
- U1 pad 2: GND -> Net-(D1-A)
- U1 pad 3: Net-(U1-VIOUT) -> Net-(D2-A)
- U1 pad 4: /A -> unconnected-(U1-PC15-Pad4)
- U2 pad 4: /C -> /A

Commit message: VER1.0: добавил драйвера и все питание схемы
Parts:
- removed R11, R12, R22, R23, R29, R30, R33, R34, R5, R6: 4.7, Resistor_SMD:R_0805_2012Metric_Pad1.20x1.40mm_HandSolder
- added C100: 56p, Capacitor_SMD:C_0603_1608Metric_Pad1.08x0.95mm_HandSolder, F.Cu at (162.8, 137.5)
- added C101: 56p, Capacitor_SMD:C_0603_1608Metric_Pad1.08x0.95mm_HandSolder, F.Cu at (165.3, 137.5)
- added C108: 10u, Capacitor_SMD:C_1206_3216Metric_Pad1.33x1.80mm_HandSolder, F.Cu at (154.5, 131.1)
- added C109: 10u, Capacitor_SMD:C_1206_3216Metric_Pad1.33x1.80mm_HandSolder, F.Cu at (157.8, 131.1)
- added C110: 10u, Capacitor_SMD:C_1206_3216Metric_Pad1.33x1.80mm_HandSolder, F.Cu at (144.4, 125.1)
- added C111: 10u, Capacitor_SMD:C_1206_3216Metric_Pad1.33x1.80mm_HandSolder, F.Cu at (147.8, 125.1)
- added C112: 10u, Capacitor_SMD:C_1206_3216Metric_Pad1.33x1.80mm_HandSolder, F.Cu at (151.1, 125.1)
- added C113: 10u, Capacitor_SMD:C_1206_3216Metric_Pad1.33x1.80mm_HandSolder, F.Cu at (154.5, 125.1)
- added C114: 10u, Capacitor_SMD:C_1206_3216Metric_Pad1.33x1.80mm_HandSolder, F.Cu at (157.8, 125.1)
- added C115: 10u, Capacitor_SMD:C_1206_3216Metric_Pad1.33x1.80mm_HandSolder, F.Cu at (144.4, 119.1)
- added C116: 10u, Capacitor_SMD:C_1206_3216Metric_Pad1.33x1.80mm_HandSolder, F.Cu at (147.8, 119.1)
- added C117: 10u, Capacitor_SMD:C_1206_3216Metric_Pad1.33x1.80mm_HandSolder, F.Cu at (151.1, 119.1)
- added C34: 56p, Capacitor_SMD:C_0603_1608Metric_Pad1.08x0.95mm_HandSolder, F.Cu at (124.5, 44.7)
- added C35: 470n, Capacitor_SMD:C_1206_3216Metric_Pad1.33x1.80mm_HandSolder, F.Cu at (124.5, 48.0)
- added C36: 470n, Capacitor_SMD:C_1206_3216Metric_Pad1.33x1.80mm_HandSolder, F.Cu at (124.5, 51.4)
- added C37: 470n, Capacitor_SMD:C_1206_3216Metric_Pad1.33x1.80mm_HandSolder, F.Cu at (124.5, 54.7)
- added C38: 470n, Capacitor_SMD:C_1206_3216Metric_Pad1.33x1.80mm_HandSolder, F.Cu at (124.5, 58.1)
- added C39: 470n, Capacitor_SMD:C_1206_3216Metric_Pad1.33x1.80mm_HandSolder, F.Cu at (124.5, 61.4)
- added C40: 470n, Capacitor_SMD:C_1206_3216Metric_Pad1.33x1.80mm_HandSolder, F.Cu at (124.5, 64.8)
- added C41: 470n, Capacitor_SMD:C_1206_3216Metric_Pad1.33x1.80mm_HandSolder, F.Cu at (130.5, 44.7)
- added C42: 470n, Capacitor_SMD:C_1206_3216Metric_Pad1.33x1.80mm_HandSolder, F.Cu at (130.5, 48.0)
- added C43: 470n, Capacitor_SMD:C_1206_3216Metric_Pad1.33x1.80mm_HandSolder, F.Cu at (130.5, 51.4)
- added C44: 10u, Capacitor_SMD:C_1206_3216Metric_Pad1.33x1.80mm_HandSolder, F.Cu at (130.5, 54.7)
- added C45: 470n, Capacitor_SMD:C_1206_3216Metric_Pad1.33x1.80mm_HandSolder, F.Cu at (130.5, 58.1)
- added C46: 470n, Capacitor_SMD:C_1206_3216Metric_Pad1.33x1.80mm_HandSolder, F.Cu at (130.5, 61.4)
- added C47: 470n, Capacitor_SMD:C_1206_3216Metric_Pad1.33x1.80mm_HandSolder, F.Cu at (130.5, 64.8)
- added C48: 470n, Capacitor_SMD:C_1206_3216Metric_Pad1.33x1.80mm_HandSolder, F.Cu at (136.5, 44.7)
- added C49: 470n, Capacitor_SMD:C_1206_3216Metric_Pad1.33x1.80mm_HandSolder, F.Cu at (49.0, 96.4)
- added C50: 470n, Capacitor_SMD:C_1206_3216Metric_Pad1.33x1.80mm_HandSolder, F.Cu at (49.0, 99.7)
- added C51: 1u, Capacitor_SMD:C_0805_2012Metric_Pad1.18x1.45mm_HandSolder, F.Cu at (72.4, 96.2)
- added C52: 100n, Capacitor_SMD:C_0805_2012Metric_Pad1.18x1.45mm_HandSolder, F.Cu at (72.4, 99.2)
- added C53: 1u, Capacitor_SMD:C_0805_2012Metric_Pad1.18x1.45mm_HandSolder, F.Cu at (72.4, 102.2)
- added C54: 100n, Capacitor_SMD:C_0805_2012Metric_Pad1.18x1.45mm_HandSolder, F.Cu at (72.4, 105.2)
- added C55: 470n, Capacitor_SMD:C_1206_3216Metric_Pad1.33x1.80mm_HandSolder, F.Cu at (49.0, 103.1)
- added C56: 470n, Capacitor_SMD:C_1206_3216Metric_Pad1.33x1.80mm_HandSolder, F.Cu at (49.0, 106.4)
- added C57: 470n, Capacitor_SMD:C_1206_3216Metric_Pad1.33x1.80mm_HandSolder, F.Cu at (49.0, 109.8)
- added C58: 470n, Capacitor_SMD:C_1206_3216Metric_Pad1.33x1.80mm_HandSolder, F.Cu at (49.0, 113.1)
- added C59: 470n, Capacitor_SMD:C_1206_3216Metric_Pad1.33x1.80mm_HandSolder, F.Cu at (49.0, 116.5)
- added C60: 470n, Capacitor_SMD:C_1206_3216Metric_Pad1.33x1.80mm_HandSolder, F.Cu at (49.0, 119.8)
- added C61: 470n, Capacitor_SMD:C_1206_3216Metric_Pad1.33x1.80mm_HandSolder, F.Cu at (49.0, 123.2)
- added C62: 470n, Capacitor_SMD:C_1206_3216Metric_Pad1.33x1.80mm_HandSolder, F.Cu at (55.0, 96.4)
- added C63: 470n, Capacitor_SMD:C_1206_3216Metric_Pad1.33x1.80mm_HandSolder, F.Cu at (55.0, 99.7)
- added C64: 470n, Capacitor_SMD:C_1206_3216Metric_Pad1.33x1.80mm_HandSolder, F.Cu at (55.0, 103.1)
- added C65: 470n, Capacitor_SMD:C_1206_3216Metric_Pad1.33x1.80mm_HandSolder, F.Cu at (55.0, 106.4)
- added C66: 10u, Capacitor_Tantalum_SMD:CP_EIA-3216-18_Kemet-A_HandSolder, F.Cu at (136.5, 48.0)
- added C67: 470n, Capacitor_SMD:C_1206_3216Metric_Pad1.33x1.80mm_HandSolder, F.Cu at (55.0, 109.8)
- added C68: 10u, Capacitor_Tantalum_SMD:CP_EIA-3216-18_Kemet-A_HandSolder, F.Cu at (136.5, 51.4)
- added C69: 10u, Capacitor_Tantalum_SMD:CP_EIA-3216-18_Kemet-A_HandSolder, F.Cu at (136.5, 54.7)
- added C70: 470n, Capacitor_SMD:C_1206_3216Metric_Pad1.33x1.80mm_HandSolder, F.Cu at (55.0, 113.1)
- added C71: 470n, Capacitor_SMD:C_1206_3216Metric_Pad1.33x1.80mm_HandSolder, F.Cu at (55.0, 116.5)
- added C72: 470n, Capacitor_SMD:C_1206_3216Metric_Pad1.33x1.80mm_HandSolder, F.Cu at (55.0, 119.8)
- added C73: 470n, Capacitor_SMD:C_1206_3216Metric_Pad1.33x1.80mm_HandSolder, F.Cu at (55.0, 123.2)
- added C74: 470n, Capacitor_SMD:C_1206_3216Metric_Pad1.33x1.80mm_HandSolder, F.Cu at (61.0, 96.4)
- added C75: 470n, Capacitor_SMD:C_1206_3216Metric_Pad1.33x1.80mm_HandSolder, F.Cu at (61.0, 99.7)
- added C76: 470n, Capacitor_SMD:C_1206_3216Metric_Pad1.33x1.80mm_HandSolder, F.Cu at (61.0, 103.1)
- added C77: 470n, Capacitor_SMD:C_1206_3216Metric_Pad1.33x1.80mm_HandSolder, F.Cu at (61.0, 106.4)
- added C78: 470n, Capacitor_SMD:C_1206_3216Metric_Pad1.33x1.80mm_HandSolder, F.Cu at (61.0, 109.8)
- added C79: 470n, Capacitor_SMD:C_1206_3216Metric_Pad1.33x1.80mm_HandSolder, F.Cu at (61.0, 113.1)
- added C80: 470n, Capacitor_SMD:C_1206_3216Metric_Pad1.33x1.80mm_HandSolder, F.Cu at (61.0, 116.5)
- added C81: 470n, Capacitor_SMD:C_1206_3216Metric_Pad1.33x1.80mm_HandSolder, F.Cu at (61.0, 119.8)
- added C82: 470n, Capacitor_SMD:C_1206_3216Metric_Pad1.33x1.80mm_HandSolder, F.Cu at (61.0, 123.2)
- added C83: 470n, Capacitor_SMD:C_1206_3216Metric_Pad1.33x1.80mm_HandSolder, F.Cu at (67.0, 96.4)
- added C84: 470n, Capacitor_SMD:C_1206_3216Metric_Pad1.33x1.80mm_HandSolder, F.Cu at (67.0, 99.7)
- added C85: 470n, Capacitor_SMD:C_1206_3216Metric_Pad1.33x1.80mm_HandSolder, F.Cu at (67.0, 103.1)
- added C86: 470n, Capacitor_SMD:C_1206_3216Metric_Pad1.33x1.80mm_HandSolder, F.Cu at (67.0, 106.4)
- added C87: 470n, Capacitor_SMD:C_1206_3216Metric_Pad1.33x1.80mm_HandSolder, F.Cu at (67.0, 109.8)
- added C88: 10u, Capacitor_SMD:C_1206_3216Metric_Pad1.33x1.80mm_HandSolder, F.Cu at (173.2, 141.0)
- added C89: 56p, Capacitor_SMD:C_0603_1608Metric_Pad1.08x0.95mm_HandSolder, F.Cu at (162.8, 141.9)
- added C90: 10u, Capacitor_SMD:C_1206_3216Metric_Pad1.33x1.80mm_HandSolder, F.Cu at (144.4, 131.1)
- added C91: 22u, Capacitor_SMD:C_1206_3216Metric_Pad1.33x1.80mm_HandSolder, F.Cu at (147.8, 131.1)
- added C92: 10u, Capacitor_SMD:C_1206_3216Metric_Pad1.33x1.80mm_HandSolder, F.Cu at (151.1, 131.1)
- added C93: 56p, Capacitor_SMD:C_0603_1608Metric_Pad1.08x0.95mm_HandSolder, F.Cu at (165.3, 141.9)
- added C94: 10u, Capacitor_SMD:C_1206_3216Metric_Pad1.33x1.80mm_HandSolder, F.Cu at (176.6, 141.0)
- added C95: 10u, Capacitor_SMD:C_1206_3216Metric_Pad1.33x1.80mm_HandSolder, F.Cu at (179.9, 141.0)
- added C96: 56p, Capacitor_SMD:C_0603_1608Metric_Pad1.08x0.95mm_HandSolder, F.Cu at (167.8, 141.9)
- added C97: 56p, Capacitor_SMD:C_0603_1608Metric_Pad1.08x0.95mm_HandSolder, F.Cu at (170.3, 141.9)
- added C98: 10u, Capacitor_SMD:C_1206_3216Metric_Pad1.33x1.80mm_HandSolder, F.Cu at (183.3, 141.0)
- added C99: 10u, Capacitor_SMD:C_1206_3216Metric_Pad1.33x1.80mm_HandSolder, F.Cu at (186.6, 141.0)
- added D10: NSD1624, Package_SO:SOIC-8_3.9x4.9mm_P1.27mm, F.Cu at (164.9, 148.3)
- added D11: D_Small, Diode_SMD:D_SMA, F.Cu at (141.8, 52.8)
- added D12: NSD1624, Package_SO:SOIC-8_3.9x4.9mm_P1.27mm, F.Cu at (171.4, 148.3)
- added D13: ~, LED_SMD:LED_0805_2012Metric, F.Cu at (133.5, 110.0)
- added D14: ~, MORNSUN:URB_S-6WR3, F.Cu at (116.2, 122.3)
- added D15: ~, LED_SMD:LED_0805_2012Metric, F.Cu at (136.5, 110.0)
- added D16: D_Small, Diode_SMD:D_SMA, F.Cu at (163.8, 126.9)
- added D17: NSD1624, Package_SO:SOIC-8_3.9x4.9mm_P1.27mm, F.Cu at (178.0, 148.3)
- added D18: D_Small, Diode_SMD:D_SMA, F.Cu at (168.3, 126.9)
- added D19: ~, Package_SO:SOIC-16_3.9x9.9mm_P1.27mm, F.Cu at (177.4, 133.8)
- added D20: ~, MORNSUN:B_S-2WR3, F.Cu at (126.4, 124.3)
- added D21: ~, MORNSUN:B_S-2WR3, F.Cu at (135.7, 124.3)
- added D23: K7815-500R3, MORNSUN:K78xx-500R3, F.Cu at (149.0, 109.4)
- added L1: L, Inductor_THT:L_Radial_D50.8mm_P38.86mm_Vishay_IHB-6, F.Cu at (286.7, 69.2)
- added L2: L, Inductor_THT:L_Radial_D50.8mm_P38.86mm_Vishay_IHB-6, F.Cu at (286.7, 121.5)
- added L3: 4.7u, Inductor_SMD:L_Taiyo-Yuden_MD-4040, F.Cu at (142.5, 59.5)
- added L4: 10u, Inductor_SMD:L_6.3x6.3_H3, F.Cu at (116.9, 148.2)
- added L5: 10u, Inductor_SMD:L_6.3x6.3_H3, F.Cu at (124.8, 148.2)
- added L6: 10u, Inductor_SMD:L_6.3x6.3_H3, F.Cu at (132.6, 148.2)
- added L7: 10u, Inductor_SMD:L_6.3x6.3_H3, F.Cu at (140.5, 148.2)
- added R52: 120, Resistor_SMD:R_0603_1608Metric_Pad0.98x0.95mm_HandSolder, F.Cu at (146.4, 52.8)
- added R53: 2k, Resistor_SMD:R_0805_2012Metric_Pad1.20x1.40mm_HandSolder, F.Cu at (77.2, 96.2)
- added R54: 3k, Resistor_SMD:R_0805_2012Metric_Pad1.20x1.40mm_HandSolder, F.Cu at (77.2, 99.1)
- added R55: 2k, Resistor_SMD:R_0805_2012Metric_Pad1.20x1.40mm_HandSolder, F.Cu at (77.2, 102.1)
- added R56: 3k, Resistor_SMD:R_0805_2012Metric_Pad1.20x1.40mm_HandSolder, F.Cu at (77.2, 105.0)
- added R57: 120, Resistor_SMD:R_0603_1608Metric_Pad0.98x0.95mm_HandSolder, F.Cu at (146.4, 55.7)
- added R58: 1k, Resistor_SMD:R_0805_2012Metric_Pad1.20x1.40mm_HandSolder, F.Cu at (133.4, 105.4)
- added R59: 1k, Resistor_SMD:R_0805_2012Metric_Pad1.20x1.40mm_HandSolder, F.Cu at (136.4, 105.4)
- added R60: 120, Resistor_SMD:R_0603_1608Metric_Pad0.98x0.95mm_HandSolder, F.Cu at (167.8, 137.5)
- added R61: 120, Resistor_SMD:R_0603_1608Metric_Pad0.98x0.95mm_HandSolder, F.Cu at (170.3, 137.5)
- added R62: 120, Resistor_SMD:R_0603_1608Metric_Pad0.98x0.95mm_HandSolder, F.Cu at (162.8, 133.2)
- added R63: 120, Resistor_SMD:R_0603_1608Metric_Pad0.98x0.95mm_HandSolder, F.Cu at (165.3, 133.2)
- added R64: 120, Resistor_SMD:R_0603_1608Metric_Pad0.98x0.95mm_HandSolder, F.Cu at (167.8, 133.2)
- added R65: 120, Resistor_SMD:R_0603_1608Metric_Pad0.98x0.95mm_HandSolder, F.Cu at (170.3, 133.2)
- added U10: AMS1117-3.3, Package_TO_SOT_SMD:SOT-223-3_TabPin2, F.Cu at (125.5, 139.0)
- added U11: AMS1117-3.3, Package_TO_SOT_SMD:SOT-223-3_TabPin2, F.Cu at (133.8, 139.0)
- added U12: NSI8220, Package_SO:SOIC-8_3.9x4.9mm_P1.27mm, F.Cu at (184.6, 148.3)
- added U6: NSI8220, Package_SO:SOIC-8_3.9x4.9mm_P1.27mm, F.Cu at (144.5, 47.2)
- added U7: CH704150CT, Sensor_Current:Allegro_CB_PFF, F.Cu at (54.4, 93.2)
- added U8: CH704150CT, Sensor_Current:Allegro_CB_PFF, F.Cu at (75.1, 93.2)
- added U9: AMS1117-5.0, Package_TO_SOT_SMD:SOT-223-3_TabPin2, F.Cu at (117.2, 139.0)
- C12, C8: value 2.2u -> 470n; footprint Capacitor_THT:C_Rect_L31.5mm_W13.0mm_P27.50mm_MKS4 -> Capacitor_SMD:C_1206_3216Metric_Pad1.33x1.80mm_HandSolder
- C31: value 10u -> 56p; footprint Capacitor_SMD:C_1206_3216Metric_Pad1.33x1.80mm_HandSolder -> Capacitor_SMD:C_0603_1608Metric_Pad1.08x0.95mm_HandSolder
- C6: value 2.2u -> 47u; footprint Capacitor_THT:C_Rect_L31.5mm_W13.0mm_P27.50mm_MKS4 -> Capacitor_THT:CP_Radial_D6.3mm_P2.50mm
- U4: value ~ -> NSI8220; footprint Package_TO_SOT_SMD:SOT-223-3_TabPin2 -> Package_SO:SOIC-8_3.9x4.9mm_P1.27mm
- moved C6 14.7 mm to (128.0, 109.4), turned to 90 degrees
Connections:
- net /A renamed /Power/A
- net /B renamed /Power/B
- net /C renamed /Power/C
- net /Current_A renamed /Power/Current_A
- net /Current_C renamed /Power/Current_C
- net /GH1 renamed /Power/GH1
- net /GH1_ON renamed /Power/GH1_ON
- net /GH2 renamed /Power/GH2
- net /GH2_ON renamed /Power/GH2_ON
- net /GH3 renamed /Power/GH3
- net /GH3_ON renamed /Power/GH3_ON
- net /GH4 renamed /Power/GH4
- net /GH4_ON renamed /Power/GH4_ON
- net /GH5 renamed /Power/GH5
- net /GL1 renamed /Power/GL1
- net /GL1_ON renamed /Power/GL1_ON
- net /GL2 renamed /Power/GL2
- net /GL2_ON renamed /Power/GL2_ON
- net /GL3 renamed /Power/GL3
- net /GL3_ON renamed /Power/GL3_ON
- net /GL4 renamed /Power/GL4
- net /GL4_ON renamed /Power/GL4_ON
- net /GL5 renamed /Power/GL5
- net /GL5_ON renamed /Power/GL5_ON
- net /S1 renamed /Power/S1
- net /S2 renamed /Power/S2
- net /Voltage_MCU renamed /Power/Voltage_MCU
- C12 pad 1: Net-(Q1-D) -> GNDPWR
- C12 pad 2: GNDPWR -> /Power/DC+
- C13 pad 2: Net-(Q1-D) -> /Power/DC+
- C16 pad 1: GNDPWR -> Net-(D3-A)
- C19 pad 2: +24V -> Net-(D7-Vin)
- C23 pad 2: +24V -> Net-(U7-IP+)
- C24 pad 2: +24V -> Net-(U8-IP+)
- C27 pad 2: +24V -> Net-(U7-IP+)
- C28 pad 2: +24V -> Net-(U8-IP+)
- C29 pad 1: +24V -> Net-(U7-IP+)
- C30 pad 1: +24V -> Net-(U8-IP+)
- C31 pad 2: +3.3VP -> Net-(D10-HI)
- C6 pad 1: Net-(Q1-D) -> +24V
- C7 pad 2: Net-(Q1-D) -> /Power/DC+
- C8 pad 1: Net-(Q1-D) -> GNDPWR
- C8 pad 2: GNDPWR -> /Power/DC+
- C9 pad 2: Net-(Q1-D) -> /Power/DC+
- D3 pad 2: GNDPWR -> Net-(D3-A)
- D4 pad 1: GNDPWR -> Net-(D3-A)
- D6 pad 3: GNDPWR -> Net-(D3-A)
- D6 pad 4: GNDPWR -> Net-(D3-A)
- D7 pad 1: +24V -> Net-(D7-Vin)
- Q1 pad 2: Net-(Q1-D) -> /Power/DC+
- Q3 pad 2: Net-(Q1-D) -> /Power/DC+
- Q5 pad 2: Net-(Q1-D) -> /Power/DC+
- Q7 pad 2: Net-(Q1-D) -> /Power/DC+
- Q8 pad 2: Net-(Q1-D) -> /Power/DC+
- R37 pad 1: /Bat_IN+ -> +24V
- R38 pad 2: /Bat_IN+ -> +24V
- R44 pad 1: GNDPWR -> Net-(D3-A)
- U4 pad 1: GNDPWR -> +3.3V
- U4 pad 2: +3.3VP -> unconnected-(U4-VIA-Pad2)
- U4 pad 3: Net-(D7-+Vo) -> unconnected-(U4-VIB-Pad3)

Commit message: VER1.0: составил список примерно 95% компонентов
Parts:
- added C102: 56p, Capacitor_SMD:C_0603_1608Metric_Pad1.08x0.95mm_HandSolder, F.Cu at (104.6, 124.8)
- added C103: 56p, Capacitor_SMD:C_0603_1608Metric_Pad1.08x0.95mm_HandSolder, F.Cu at (104.6, 127.3)
- added C104: 10u, Capacitor_SMD:C_1206_3216Metric_Pad1.33x1.80mm_HandSolder, F.Cu at (97.0, 136.8)
- added C105: 10u, Capacitor_SMD:C_1206_3216Metric_Pad1.33x1.80mm_HandSolder, F.Cu at (97.0, 140.1)
- added C106: 10p, Capacitor_SMD:C_0805_2012Metric_Pad1.18x1.45mm_HandSolder, F.Cu at (84.4, 125.0)
- added C107: 10p, Capacitor_SMD:C_0805_2012Metric_Pad1.18x1.45mm_HandSolder, F.Cu at (84.4, 128.0)
- added C118: 2.2u, Capacitor_SMD:C_0805_2012Metric_Pad1.18x1.45mm_HandSolder, F.Cu at (84.4, 131.0)
- added C119: 100n, Capacitor_SMD:C_0805_2012Metric_Pad1.18x1.45mm_HandSolder, F.Cu at (84.4, 134.0)
- added C120: 2.2u, Capacitor_SMD:C_0805_2012Metric_Pad1.18x1.45mm_HandSolder, F.Cu at (84.4, 137.0)
- added C121: 100n, Capacitor_SMD:C_0805_2012Metric_Pad1.18x1.45mm_HandSolder, F.Cu at (84.4, 140.1)
- added C122: 100n, Capacitor_SMD:C_0805_2012Metric_Pad1.18x1.45mm_HandSolder, F.Cu at (84.4, 143.1)
- added C123: 100n, Capacitor_SMD:C_0805_2012Metric_Pad1.18x1.45mm_HandSolder, F.Cu at (84.4, 146.1)
- added C124: 100n, Capacitor_SMD:C_0805_2012Metric_Pad1.18x1.45mm_HandSolder, F.Cu at (102.4, 136.6)
- added C125: 100n, Capacitor_SMD:C_0805_2012Metric_Pad1.18x1.45mm_HandSolder, F.Cu at (102.4, 139.6)
- added C126: 100n, Capacitor_SMD:C_0805_2012Metric_Pad1.18x1.45mm_HandSolder, F.Cu at (109.9, 124.0)
- added C127: 100n, Capacitor_SMD:C_0805_2012Metric_Pad1.18x1.45mm_HandSolder, F.Cu at (109.9, 127.0)
- added C128: 100n, Capacitor_SMD:C_0805_2012Metric_Pad1.18x1.45mm_HandSolder, F.Cu at (109.9, 130.0)
- added C129: 100n, Capacitor_SMD:C_0805_2012Metric_Pad1.18x1.45mm_HandSolder, F.Cu at (109.9, 133.0)
- added C130: 100n, Capacitor_SMD:C_0805_2012Metric_Pad1.18x1.45mm_HandSolder, F.Cu at (109.9, 136.0)
- added C131: 100n, Capacitor_SMD:C_0805_2012Metric_Pad1.18x1.45mm_HandSolder, F.Cu at (109.9, 139.1)
- added D22: ~, Package_SO:SOIC-16_3.9x9.9mm_P1.27mm, F.Cu at (98.2, 129.4)
- added D41: ~, Package_TO_SOT_SMD:SOT-23, F.Cu at (89.3, 135.0)
- added D42: ~, Package_TO_SOT_SMD:SOT-23, F.Cu at (89.3, 139.4)
- added R66: 120, Resistor_SMD:R_0603_1608Metric_Pad0.98x0.95mm_HandSolder, F.Cu at (104.6, 129.8)
- added R67: 120, Resistor_SMD:R_0603_1608Metric_Pad0.98x0.95mm_HandSolder, F.Cu at (104.6, 132.3)
- added R81: 100, Resistor_SMD:R_0805_2012Metric_Pad1.20x1.40mm_HandSolder, F.Cu at (74.9, 125.0)
- added R82: 0, Resistor_SMD:R_0805_2012Metric_Pad1.20x1.40mm_HandSolder, F.Cu at (74.9, 127.9)
- added R83: 0, Resistor_SMD:R_0805_2012Metric_Pad1.20x1.40mm_HandSolder, F.Cu at (74.9, 130.9)
- added R84: 1k, Resistor_SMD:R_0805_2012Metric_Pad1.20x1.40mm_HandSolder, F.Cu at (74.9, 133.8)
- added R85: 1k, Resistor_SMD:R_0805_2012Metric_Pad1.20x1.40mm_HandSolder, F.Cu at (74.9, 136.8)
- added R87: 100, Resistor_SMD:R_0805_2012Metric_Pad1.20x1.40mm_HandSolder, F.Cu at (74.9, 139.7)
- added R88: 0, Resistor_SMD:R_0805_2012Metric_Pad1.20x1.40mm_HandSolder, F.Cu at (79.6, 125.0)
- added R89: 0, Resistor_SMD:R_0805_2012Metric_Pad1.20x1.40mm_HandSolder, F.Cu at (79.6, 127.9)
- added R90: 1k, Resistor_SMD:R_0805_2012Metric_Pad1.20x1.40mm_HandSolder, F.Cu at (79.6, 130.9)
- added R91: 1k, Resistor_SMD:R_0805_2012Metric_Pad1.20x1.40mm_HandSolder, F.Cu at (79.6, 133.8)
- added U19: ~, Package_TO_SOT_SMD:SOT-23-6, F.Cu at (89.4, 125.9)
- added U20: ~, Package_TO_SOT_SMD:SOT-23-6, F.Cu at (89.4, 130.5)
- C12, C13, C35, C36, C37, C38, C39, C40, C41, C42, C43, C45, C46, C47, C48, C49, C50, C55, C56, C57, C58, C59, C60, C61, C62, C63, C64, C65, C67, C7, C70, C71, C72, C73, C74, C75, C76, C77, C78, C79, C8, C80, C81, C82, C83, C84, C85, C86, C87, C9: footprint Capacitor_SMD:C_1206_3216Metric_Pad1.33x1.80mm_HandSolder -> Capacitor_SMD:C_1210_3225Metric_Pad1.33x2.70mm_HandSolder
- D10, D12, D17: value NSD1624 -> ~
- D11, D16, D18: value D_Small -> ~
- D23: value K7815-500R3 -> ~
- D7: value K7805-500R3 -> ~
- Q1, Q10, Q2, Q3, Q4, Q5, Q6, Q7, Q8, Q9: value WMK115N15HG2 -> ~
- U1: value STM32F405RGTx -> ~
- U10, U11: value AMS1117-3.3 -> ~
- U12, U4, U6: value NSI8220 -> ~
- U2, U3, U7, U8: value CH704150CT -> ~
- U9: value AMS1117-5.0 -> ~
Connections:
- C23 pad 2: Net-(U7-IP+) -> +24V
- C24 pad 2: Net-(U8-IP+) -> +24V
- C27 pad 2: Net-(U7-IP+) -> +24V
- C28 pad 2: Net-(U8-IP+) -> +24V
- C29 pad 1: Net-(U7-IP+) -> +24V
- C30 pad 1: Net-(U8-IP+) -> +24V
- L1 pad 1: /Power/S1 -> Net-(U7-IP-)
- L1 pad 2: Net-(U7-IP+) -> +24V
- L2 pad 1: /Power/S2 -> Net-(U8-IP-)
- L2 pad 2: Net-(U8-IP+) -> +24V
- U7 pad 4: Net-(U7-IP+) -> /Power/S1
- U7 pad 5: +24V -> Net-(U7-IP-)
- U8 pad 4: Net-(U8-IP+) -> /Power/S2
- U8 pad 5: +24V -> Net-(U8-IP-)
