File: Nauka_DCAC.kicad_sch (KiCad schematic)
At the start: 84 parts, among them J1 Conn_01x01, J2 Conn_01x01, J3 Conn_01x01, J4 Conn_01x01, J5 Conn_01x01, Q1 WMK115N15HG2, Q2 WMK115N15HG2, Q3 WMK115N15HG2, Q4 WMK115N15HG2, Q5 WMK115N15HG2, Q6 WMK115N15HG2, Q7 WMK115N15HG2, Q8 WMK115N15HG2, U1 CH704150CT, U2 CH704150CT

Commit message: VER1.0: собрал силовую часть на схеме
Parts:
- removed C2: C, symbol Device:C
- added C1, C2: 12p, Capacitor_SMD:C_0805_2012Metric_Pad1.18x1.45mm_HandSolder, symbol Device:C_Small
- added C13, C7, C9: 470n, Capacitor_SMD:C_1206_3216Metric_Pad1.33x1.80mm_HandSolder, symbol Device:C_Small
- added C23, C24, C27, C28: 2.2u, Capacitor_SMD:C_1206_3216Metric_Pad1.33x1.80mm_HandSolder, symbol Device:C_Small
- added C29, C30: 1m, Capacitor_THT:CP_Radial_D16.0mm_P7.50mm, symbol Device:C_Polarized
- added C3: 100n, Capacitor_SMD:C_0805_2012Metric_Pad1.18x1.45mm_HandSolder, symbol Device:C_Small
- added C4, C5: 2.2u, Capacitor_SMD:C_0805_2012Metric_Pad1.18x1.45mm_HandSolder, symbol Device:C_Small
- added C6, C8: 2.2u, Capacitor_THT:C_Rect_L31.5mm_W13.0mm_P27.50mm_MKS4, symbol Device:C
- added D1, D2: (no value), LED_SMD:LED_0805_2012Metric, symbol Device:LED_Small
- added L1: L, symbol Device:L
- added Q7, Q9: WMK115N15HG2, Package_TO_SOT_THT:TO-220-3_Horizontal_TabUp, symbol Transistor_FET:BUZ11
- added R15, R24, R25, R28: 10k, Resistor_SMD:R_0805_2012Metric_Pad1.20x1.40mm_HandSolder, symbol Device:R_Small
- added R16, R21: 1k, Resistor_SMD:R_0805_2012Metric_Pad1.20x1.40mm_HandSolder, symbol Device:R_Small
- added R31, R32: 10, Resistor_SMD:R_0805_2012Metric_Pad1.20x1.40mm_HandSolder, symbol Device:R_Small
- added R33, R34: 4.7, Resistor_SMD:R_0805_2012Metric_Pad1.20x1.40mm_HandSolder, symbol Device:R_Small
- added U1: STM32F405RGTx, Package_QFP:LQFP-64_10x10mm_P0.5mm, symbol MCU_ST_STM32F4:STM32F405RGTx
- added Y1: 16M, Crystal:Crystal_SMD_SeikoEpson_FA238-4Pin_3.2x2.5mm, symbol Device:Crystal_GND24
- C12: renamed from C1; value C -> 2.2u; footprint (none) -> Capacitor_THT:C_Rect_L31.5mm_W13.0mm_P27.50mm_MKS4
- renumbered C4 to C10, C3 to C11, C5 to C14, C6 to C15, C7 to C16, C14 to C17, C15 to C18, C77 to C19, C13 to C20, C12 to C21, C76 to C22, C8 to C25, C9 to C26, C83 to C31, C10 to C32, C11 to C33, D33 to D3, D32 to D4, D35 to D5, D36 to D6, D1 to D7, D37 to D8, D38 to D9, L1 to L2, Q7 to Q1, Q2 to Q10, Q8 to Q2, Q5 to Q3, Q6 to Q4, Q4 to Q5, Q3 to Q6, Q1 to Q8, R5 to R1, R21 to R10, R16 to R11, R22 to R12, R7 to R13, R3 to R14, R8 to R17, R4 to R18, R17 to R19, R1 to R2, R23 to R20, R18 to R22, R24 to R23, R25 to R26, R26 to R27, R27 to R29, R13 to R3, R28 to R30, R9 to R35, R10 to R36, R65 to R37, R66 to R38, R11 to R39, R19 to R4, R12 to R40, R67 to R41, R68 to R42, R69 to R43, R70 to R44, R29 to R45, R30 to R46, R31 to R47, R32 to R48, R33 to R49, R14 to R5, R74 to R50, R34 to R51, R20 to R6, R6 to R7, R2 to R8, R15 to R9, U1 to U2, U2 to U3, U32 to U4, U16 to U5
Connections:
- net Bat_IN+ is gone; now on net +24V: R37.1, R38.2
- net +24V: now also C23.2, C24.2, C27.2, C28.2, C29.1, C30.1, L1.2
- net +3.3V: now also R28.1, U1.1 (VBAT), U1.13 (VDDA), U1.19 (VDD), U1.32 (VDD), U1.48 (VDD), U1.64 (VDD)
- net GH4: now also Q7.1 (G); no longer Q8.1 (G)
- net GH4_OFF: now also R33.2
- net GH4_ON: now also R31.2
- net GL3: no longer R27.1, R30.1
- net GL4: now also R27.1, R30.1, Q9.1 (G); no longer Q10.1 (G)
- net GND: now also C1.1, C2.2, C3.1, C4.2, C5.2, R15.1, R16.2, R21.2, U1.12 (VSSA), U1.18 (VSS), U1.63 (VSS), Y1.2, Y1.4
- net GNDPWR: now also C13.1, C23.1, C24.1, C27.1, C28.1, C29.2, C30.2, C6.2, C7.1, C8.2, C9.1, Q9.3 (S), R25.2
- net at C12.1, Q1.2 (D), Q3.2 (D)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: now also C13.2, C6.1, C7.2, C8.1, C9.2, Q7.2 (D)
- net Bat+ renamed S2
- net S2: now also R24.2; no longer R17.2
- new net: C2.1, U1.6 (PH1), Y1.1
- new net: C1.2, U1.5 (PH0), Y1.3
- new net: D1.2 (A), U1.2 (PC13)
- new net: D2.2 (A), U1.3 (PC14)
- new net: C4.1, U1.31 (VCAP_1)
- new net: C5.1, U1.47 (VCAP_2)
- new net: D2.1 (K), R21.1
- new net: D1.1 (K), R16.1
- new net BOOT: R15.2, U1.60 (BOOT0)
- new net GH5: Q8.1 (G), R24.1, R31.1, R33.1
- new net GL5: Q10.1 (G), R25.1, R32.1, R34.1
- new net GL5_OFF: R34.2
- new net GL5_ON: R32.2
- new net NRST: C3.2, R28.2, U1.7 (NRST)
- new net S1: L1.1, Q7.3 (S), Q9.2 (D), R17.2
Other:
- note added: "Силовая часть"
- moved on the sheet: C10, C11, C12, C14, C15, C16, C17, C18, C19, C20, C21, C22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

Commit message: VER1.0: добавил драйвера и все питание схемы
Parts:
- removed C10, C14: 1u, Capacitor_SMD:C_0805_2012Metric_Pad1.18x1.45mm_HandSolder, symbol Device:C_Small
- removed C11, C15, C18, C21, C32: 100n, Capacitor_SMD:C_0805_2012Metric_Pad1.18x1.45mm_HandSolder, symbol Device:C_Small
- removed C12, C6, C8: 2.2u, Capacitor_THT:C_Rect_L31.5mm_W13.0mm_P27.50mm_MKS4, symbol Device:C
- removed C13, C7, C9: 470n, Capacitor_SMD:C_1206_3216Metric_Pad1.33x1.80mm_HandSolder, symbol Device:C_Small
- removed C16, C25, C26: 56p, Capacitor_SMD:C_0805_2012Metric_Pad1.18x1.45mm_HandSolder, symbol Device:C_Small
- removed C17, C20: 2.2u, Capacitor_SMD:C_0805_2012Metric_Pad1.18x1.45mm_HandSolder, symbol Device:C_Small
- removed C19, C22, C31: 10u, Capacitor_SMD:C_1206_3216Metric_Pad1.33x1.80mm_HandSolder, symbol Device:C_Small
- removed C23, C24, C27, C28: 2.2u, Capacitor_SMD:C_1206_3216Metric_Pad1.33x1.80mm_HandSolder, symbol Device:C_Small
- removed C29, C30: 1m, Capacitor_THT:CP_Radial_D16.0mm_P7.50mm, symbol Device:C_Polarized
- removed C33: 1n, Capacitor_SMD:C_0805_2012Metric_Pad1.18x1.45mm_HandSolder, symbol Device:C_Small
- removed D3, D4: (no value), LED_SMD:LED_1206_3216Metric_Pad1.42x1.75mm_HandSolder, symbol Device:LED_Small
- removed D5, D9: (no value), Package_TO_SOT_SMD:SOT-23, symbol Device:D_Dual_Series_AKC_Parallel
- removed D6: (no value), Package_SO:SOIC-8_7.5x5.85mm_P1.27mm, symbol NOVSENSE:NSI1311
- removed D7: K7805-500R3, MORNSUN:K78xx-500R3, symbol MORNSUN_my:K78xx-500R3
- removed D8: (no value), LED_SMD:LED_0805_2012Metric, symbol Device:LED_Small
- removed J1, J2, J3, J4, J5: Conn_01x01, symbol Connector_Generic:Conn_01x01
- removed L1, L2: L, symbol Device:L
- removed Q1, Q10, Q2, Q3, Q4, Q5, Q6, Q7, Q8, Q9: WMK115N15HG2, Package_TO_SOT_THT:TO-220-3_Horizontal_TabUp, symbol Transistor_FET:BUZ11
- removed R1, R13, R14, R17, R18, R2, R24, R25, R7, R8: 10k, Resistor_SMD:R_0805_2012Metric_Pad1.20x1.40mm_HandSolder, symbol Device:R_Small
- removed R10, R19, R20, R26, R27, R3, R31, R32, R4, R9: 10, Resistor_SMD:R_0805_2012Metric_Pad1.20x1.40mm_HandSolder, symbol Device:R_Small
- removed R11, R12, R22, R23, R29, R30, R33, R34, R5, R6: 4.7, Resistor_SMD:R_0805_2012Metric_Pad1.20x1.40mm_HandSolder, symbol Device:R_Small
- removed R35, R39: 2k, Resistor_SMD:R_0805_2012Metric_Pad1.20x1.40mm_HandSolder, symbol Device:R_Small
- removed R36, R40: 3k, Resistor_SMD:R_0805_2012Metric_Pad1.20x1.40mm_HandSolder, symbol Device:R_Small
- removed R37: 10k, Resistor_SMD:R_1206_3216Metric_Pad1.30x1.75mm_HandSolder, symbol Device:R
- removed R38, R41, R42, R43: 110k, Resistor_SMD:R_1206_3216Metric, symbol Device:R
- removed R44: 11.3k, Resistor_SMD:R_1206_3216Metric, symbol Device:R
- removed R45: 120, Resistor_SMD:R_0805_2012Metric_Pad1.20x1.40mm_HandSolder, symbol Device:R_Small
- removed R46, R47, R48, R49: 1k, Resistor_SMD:R_0805_2012Metric_Pad1.20x1.40mm_HandSolder, symbol Device:R_Small
- removed R50: 750, Resistor_SMD:R_0805_2012Metric_Pad1.20x1.40mm_HandSolder, symbol Device:R_Small
- removed R51: 510, Resistor_SMD:R_0805_2012Metric_Pad1.20x1.40mm_HandSolder, symbol Device:R_Small
- removed U2, U3: CH704150CT, Sensor_Current:Allegro_CB_PFF, symbol Sensor_Current:ACS756xCB-100B-PFF
- removed U4: (no value), Package_TO_SOT_SMD:SOT-223-3_TabPin2, symbol Regulator_Linear:LM1117MP-3.3
- removed U5: (no value), Package_TO_SOT_SMD:SOT-23-5, symbol Amplifier_Operational:OPA333xxDBV
- added C106, C107: 10p, Capacitor_SMD:C_0805_2012Metric_Pad1.18x1.45mm_HandSolder, symbol Device:C_Small
- added C118, C120: 2.2u, Capacitor_SMD:C_0805_2012Metric_Pad1.18x1.45mm_HandSolder, symbol Device:C_Small
- added C119, C121, C122, C123: 100n, Capacitor_SMD:C_0805_2012Metric_Pad1.18x1.45mm_HandSolder, symbol Device:C_Small
- added D41, D42: (no value), Package_TO_SOT_SMD:SOT-23, symbol Device:D_Dual_Series_AKC_Parallel
- added R81, R87: 100, Resistor_SMD:R_0805_2012Metric_Pad1.20x1.40mm_HandSolder, symbol Device:R_Small
- added R82, R83, R88, R89: 0, Resistor_SMD:R_0805_2012Metric_Pad1.20x1.40mm_HandSolder, symbol Device:R_Small
- added R84, R85, R90, R91: 1k, Resistor_SMD:R_0805_2012Metric_Pad1.20x1.40mm_HandSolder, symbol Device:R_Small
- added U19, U20: TLV3501AIDBV, Package_TO_SOT_SMD:SOT-23-6, symbol Comparator:TLV3501AIDBV
Connections:
- net +3.3V: now also C118.1, C119.1, C120.1, C121.1, D41.2 (K), D42.2 (K), R84.1, R90.1, U19.4 (V+), U20.4 (V+)
- net GND: now also C106.2, C107.2, C118.2, C119.2, C120.2, C121.2, C122.2, C123.2, D41.1 (A), D42.1 (A), R82.1, R85.2, R88.1, R91.2, U19.2 (V-), U20.2 (V-)
- new net: C122.1, R83.2, R84.2, R85.1, U19.1 (-)
- new net: R81.2, U19.5
- new net: C123.1, R89.2, R90.2, R91.1, U20.1 (-)
- new net: R87.2, U20.5
- new net Current_buck_1: U19.3 (+)
- new net Current_buck_2: U20.3 (+)
- new net DAC1: R83.1
- new net DAC2: R89.1
- new net OverCurrent1: C106.1, D41.3 (common), R81.1
- new net OverCurrent2: C107.1, D42.3 (common), R87.1
- new net SHDN_OverCurrent_1: R82.2, U19.6 (SHDN)
- new net SHDN_OverCurrent_2: R88.2, U20.6 (SHDN)
Other:
- added sheet Drivers (Drivers.kicad_sch)
- added sheet Power (Power.kicad_sch)
- added sheet Supply (Supply.kicad_sch)
- note removed: "Затворные резисторы"
- note removed: "Подтяжки затворов"
- note removed: "Силовая часть"
- moved on the sheet: C1, C2, C3, C4, C5, D1, D2, R15, R16, R21, R28, U1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

Commit message: VER1.0: составил список примерно 95% компонентов
Parts:
- C1, C2, C3, C4, C5: Description P/N Capacitor SMD 50V -> Capacitor SMD 25V
- C106, C107, C118, C119, C120, C121, C122, C123: Description P/N (none) -> Capacitor SMD 25V
- R15, R16, R21, R28: Description P/N Resistor SMD -> Resistor SMD 1%
- R81, R82, R83, R84, R85, R87, R88, R89, R90, R91: Description P/N (none) -> Resistor SMD 1%
- U1: value STM32F405RGTx -> (none); Description P/N (none) -> MCU; Product Name (none) -> STM32F405RGTx
- U19, U20: value TLV3501AIDBV -> (none); Description P/N (none) -> Comparator; Product Name (none) -> TLV3501AIDBV
Changed lines of the file:
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@@
 			)
 		)
-		(property "Description P/N" ""
+		(property "Description P/N" "Resistor SMD 1%"
 			(at 237.49 191.77 0)
 			(hide yes)
@@
 			)
 		)
-		(property "Description P/N" ""
+		(property "Description P/N" "Resistor SMD 1%"
 			(at 205.74 176.53 0)
 			(hide yes)
@@
 			)
 		)
-		(property "Description P/N" ""
+		(property "Description P/N" "Capacitor SMD 25V"
 			(at 238.76 158.75 0)
 			(hide yes)
@@
 			)
 		)
-		(property "Description P/N" ""
+		(property "Description P/N" "Resistor SMD 1%"
 			(at 237.49 242.57 0)
 			(hide yes)
@@
 			)
 		)
-		(property "Description P/N" ""
+		(property "Description P/N" "Capacitor SMD 25V"
 			(at 242.57 246.38 0)
 			(hide yes)
@@
 			)
 		)
-		(property "Description P/N" ""
+		(property "Description P/N" "Resistor SMD 1%"
 			(at 205.74 227.33 0)
 			(hide yes)
@@
 			)
 		)
-		(property "Value" "STM32F405RGTx"
+		(property "Value" ""
 			(at 87.2333 125.73 0)
 			(show_name no)
@@
 			)
 		)
-		(property "Datasheet" "https://www.st.com/resource/en/datasheet/stm32f405rg.pdf"
+		(property "Datasheet" ""
 			(at 82.55 74.93 0)
 			(hide yes)
@@
 			)
 		)
+		(property "Product Name" "STM32F405RGTx"
+			(at 82.55 74.93 0)
+			(hide yes)
+			(show_name no)
+			(do_not_autoplace no)
+			(effects
+				(font
+					(size 1.27 1.27)
+				)
+			)
+		)
+		(property "Description P/N" "MCU"
+			(at 82.55 74.93 0)
+			(hide yes)
+			(show_name no)
+			(do_not_autoplace no)
+			(effects
+				(font
+					(size 1.27 1.27)
+				)
+			)
+		)
+		(property "Function" ""
+			(at 82.55 74.93 0)
+			(hide yes)
+			(show_name no)
+			(do_not_autoplace no)
+			(effects
+				(font
+					(size 1.27 1.27)
+				)
+			)
+		)
+		(property "Replacement" ""
+			(at 82.55 74.93 0)
+			(hide yes)
+			(show_name no)
+			(do_not_autoplace no)
+			(effects
+				(font
+					(size 1.27 1.27)
+				)
+			)
+		)
 		(pin "17"
 		)
@@
 			)
 		)
-		(property "Description P/N" ""
+		(property "Description P/N" "Capacitor SMD 25V"
 			(at 242.57 195.58 0)
 			(hide yes)
@@
 			)
 		)
-		(property "Description P/N" "Capacitor SMD 50V"
+		(property "Description P/N" "Capacitor SMD 25V"
 			(at 25.4 36.83 0)
 			(hide yes)
@@
 			)
 		)
-		(property "Description P/N" "Resistor SMD"
+		(property "Description P/N" "Resistor SMD 1%"
 			(at 44.45 107.95 0)
 			(hide yes)
@@
 			)
 		)
-		(property "Description P/N" ""
+		(property "Description P/N" "Capacitor SMD 25V"
 			(at 191.77 232.41 0)
 			(hide yes)
@@
 			)
 		)
-		(property "Description P/N" "Resistor SMD"
+		(property "Description P/N" "Resistor SMD 1%"
 			(at 36.83 107.95 0)
 			(hide yes)
@@
 			)
 		)
-		(property "Description P/N" ""
+		(property "Description P/N" "Resistor SMD 1%"
 			(at 251.46 238.76 0)
 			(hide yes)
@@
 			)
 		)
-		(property "Description P/N" "Capacitor SMD 50V"
+		(property "Description P/N" "Capacitor SMD 25V"
 			(at 59.69 107.95 0)
 			(hide yes)
@@
 			)
 		)
-		(property "Description P/N" "Capacitor SMD 50V"
+		(property "Description P/N" "Capacitor SMD 25V"
 			(at 52.07 29.21 0)
 			(hide yes)
@@
 			)
 		)
-		(property "Description P/N" ""
+		(property "Description P/N" "Capacitor SMD 25V"
 			(at 238.76 209.55 0)
 			(hide yes)
@@
 			)
 		)
-		(property "Description P/N" ""
+		(property "Description P/N" "Resistor SMD 1%"
 			(at 251.46 187.96 0)
 			(hide yes)
@@
 			)
 		)
-		(property "Description P/N" ""
+		(property "Description P/N" "Capacitor SMD 25V"
 			(at 238.76 217.17 0)
 			(hide yes)
@@
 			)
 		)
-		(property "Value" "TLV3501AIDBV"
+		(property "Value" ""
 			(at 217.17 223.4498 0)
 			(hide yes)
@@
 			)
 		)
-		(property "Datasheet" "https://www.ti.com/lit/ds/symlink/tlv3501.pdf"
+		(property "Datasheet" ""
 			(at 229.87 238.76 0)
 			(hide yes)
@@
 			)
 		)
+		(property "Product Name" "TLV3501AIDBV"
+			(at 229.87 227.33 0)
+			(hide yes)
+			(show_name no)
+			(do_not_autoplace no)
+			(effects
+				(font
+					(size 1.27 1.27)
+				)
+			)
+		)
+		(property "Description P/N" "Comparator"
+			(at 229.87 227.33 0)
+			(hide yes)
+			(show_name no)
+			(do_not_autoplace no)
+			(effects
+				(font
+					(size 1.27 1.27)
+				)
+			)
+		)
 		(pin "4"
 		)
@@
 			)
 		)
-		(property "Description P/N" ""
+		(property "Description P/N" "Resistor SMD 1%"
 			(at 205.74 184.15 0)
 			(hide yes)
@@
 			)
 		)
-		(property "Description P/N" "Resistor SMD"
+		(property "Description P/N" "Resistor SMD 1%"
 			(at 36.83 29.21 0)
 			(hide yes)
@@
 			)
 		)
-		(property "Value" "TLV3501AIDBV"
+		(property "Value" ""
 			(at 217.17 172.6498 0)
 			(hide yes)
@@
 			)
 		)
-		(property "Datasheet" "https://www.ti.com/lit/ds/symlink/tlv3501.pdf"
+		(property "Datasheet" ""
 			(at 229.87 187.96 0)
 			(hide yes)
@@
 			)
 		)
+		(property "Product Name" "TLV3501AIDBV"
+			(at 229.87 176.53 0)
+			(hide yes)
+			(show_name no)
+			(do_not_autoplace no)
+			(effects
+				(font
+					(size 1.27 1.27)
+				)
+			)
+		)
+		(property "Description P/N" "Comparator"
+			(at 229.87 176.53 0)
+			(hide yes)
+			(show_name no)
+			(do_not_autoplace no)
+			(effects
+				(font
+					(size 1.27 1.27)
+				)
+			)
+		)
 		(pin "4"
 		)
@@
 			)
 		)
-		(property "Description P/N" "Capacitor SMD 50V"
+		(property "Description P/N" "Capacitor SMD 25V"
 			(at 52.07 107.95 0)
 			(hide yes)
@@
 			)
 		)
-		(property "Description P/N" "Resistor SMD"
+		(property "Description P/N" "Resistor SMD 1%"
 			(at 58.42 29.21 0)
 			(hide yes)
@@
 			)
 		)
-		(property "Description P/N" ""
+		(property "Description P/N" "Resistor SMD 1%"
 			(at 251.46 195.58 0)
 			(hide yes)
@@
 			)
 		)
-		(property "Description P/N" ""
+		(property "Description P/N" "Capacitor SMD 25V"
 			(at 191.77 181.61 0)
 			(hide yes)
@@
 			)
 		)
+		(property "Function" ""
+			(at 191.77 181.61 0)
+			(hide yes)
+			(show_name no)
+			(do_not_autoplace no)
+			(effects
+				(font
+					(size 1.27 1.27)
+				)
+			)
+		)
 		(pin "1"
 		)
@@
 			)
 		)
-		(property "Description P/N" ""
+		(property "Description P/N" "Resistor SMD 1%"
 			(at 251.46 246.38 0)
 			(hide yes)
@@
 			)
 		)
-		(property "Description P/N" ""
+		(property "Description P/N" "Capacitor SMD 25V"
 			(at 238.76 166.37 0)
 			(hide yes)
@@
 			)
 		)
-		(property "Description P/N" ""
+		(property "Description P/N" "Resistor SMD 1%"
 			(at 205.74 234.95 0)
 			(hide yes)
@@
 			)
 		)
-		(property "Description P/N" "Capacitor SMD 50V"
+		(property "Description P/N" "Capacitor SMD 25V"
 			(at 25.4 54.61 0)
 			(hide yes)
