File: Power.kicad_sch (KiCad schematic)
At the start: 140 parts, among them J1 Conn_01x01, J2 Conn_01x01, J3 Conn_01x01, J4 Conn_01x01, J5 Conn_01x01, Q1 WMK115N15HG2, Q10 WMK115N15HG2, Q2 WMK115N15HG2, Q3 WMK115N15HG2, Q4 WMK115N15HG2, Q5 WMK115N15HG2, Q6 WMK115N15HG2, Q7 WMK115N15HG2, Q8 WMK115N15HG2, Q9 WMK115N15HG2, U2 CH704150CT, U3 CH704150CT, U7 CH704150CT, U8 CH704150CT

Commit message: VER1.0: составил список примерно 95% компонентов
Parts:
- C10, C11, C14, C15, C16, C17, C18, C20, C21, C25, C26, C32, C33, C51, C52, C53, C54: Description P/N (none) -> Capacitor SMD 25V
- C12, C13, C35, C36, C37, C38, C39, C40, C41, C42, C43, C45, C46, C47, C48, C49, C50, C55, C56, C57, C58, C59, C60, C61, C62, C63, C64, C65, C67, C7, C70, C71, C72, C73, C74, C75, C76, C77, C78, C79, C8, C80, C81, C82, C83, C84, C85, C86, C87, C9: footprint Capacitor_SMD:C_1206_3216Metric_Pad1.33x1.80mm_HandSolder -> Capacitor_SMD:C_1210_3225Metric_Pad1.33x2.70mm_HandSolder; Description P/N (none) -> Capacitor SMD 200V; Product Name (none) -> 1210B474K201CT
- C23, C24, C27, C28: Description P/N (none) -> Capacitor SMD 50V
- C29, C30: Description P/N (none) -> Capacitor electrolytic low ESR; Product Name (none) -> EXR102M63B
- J1, J2, J3, J4, J5: value Conn_01x01 -> (none)
- L1, L2: now left out of the parts list
- Q1, Q10, Q2, Q3, Q4, Q5, Q6, Q7, Q8, Q9: value WMK115N15HG2 -> (none); Description P/N (none) -> MOSFET; Product Name (none) -> WMK115N15HG2
- R1, R10, R13, R14, R17, R18, R19, R2, R20, R24, R25, R26, R27, R3, R31, R32, R4, R45, R46, R47, R48, R49, R51, R7, R8, R9: Description P/N (none) -> Resistor SMD 1%
- R35, R36, R39, R40, R53, R54, R55, R56: Description P/N (none) -> Resistor SMD 0.1%
- R37: Description P/N Resistor SMD -> Resistor SMD 1%
- R38, R41, R42, R43, R44: Description P/N Resistor SMD -> Resistor SMD 0.1%
- U2, U3, U7, U8: value CH704150CT -> (none); Description P/N (none) -> Current sensor; Product Name (none) -> CH704150CT
