File: Supply.kicad_sch (KiCad schematic)
At the start: 38 parts, among them U10 AMS1117-3.3, U11 AMS1117-3.3, U9 AMS1117-5.0

Commit message: VER1.0: составил список примерно 95% компонентов
Parts:
- C110, C111, C112, C115, C90, C91, C92: Description P/N (none) -> Capacitor SMD 50V
- C6: Description P/N (none) -> Capacitor electrolytic low ESR; Product Name (none) -> EEUFR1J470
- C66, C68, C69: Description P/N (none) -> Capacitor tantalum SMD 10V
- D14: Description P/N (none) -> DC/DC; Product Name (none) -> URB_S-6WR3
- D20, D21: Description P/N (none) -> DC/DC; Product Name (none) -> B2415S-2WR3
- D23: value K7815-500R3 -> (none); Description P/N (none) -> DC/DC; Product Name (none) -> K7815-500R3
- D7: value K7805-500R3 -> (none); Description P/N (none) -> DC/DC; Product Name (none) -> K7805-500R3
- L3: Description P/N (none) -> Inductor SMD; Product Name (none) -> LQH44PN4R7MP0L
- L4, L5, L6, L7: Description P/N (none) -> Inductor SMD; Product Name (none) -> LQH66SN100M03L
- R50: Description P/N Resistor SMD -> Resistor SMD 1%
- R58, R59: Description P/N (none) -> Resistor SMD 1%
- U10, U11: value AMS1117-3.3 -> (none); Description P/N (none) -> Linear regulator; Product Name (none) -> AMS1117-3.3
- U9: value AMS1117-5.0 -> (none); Description P/N (none) -> Linear regulator; Product Name (none) -> AMS1117-5.0
Other:
- moved on the sheet: C112, C113, C114, C115, C116, C117, D20, D21, L6, L7
